Commit message: add mass

File: ros_ws/src/description/urdf/description.urdf (robot description, URDF)
Before this commit: robot description, 8 links, 7 joints
Links:
- link steering_f_l: mass 0 -> 0.004
- link steering_f_r: mass 0 -> 0.004
Joints:
- removed joint steering_f_l
- removed joint steering_f_r
- removed joint tire_f_l
- removed joint tire_f_r
- removed joint tire_r_l
- removed joint tire_r_r
- added joint j_steering_f_l: type revolute, parent base_link, child steering_f_l, origin xyz=0.1135 0.07475 0 rpy=0 -0.087266 0, axis 0 0 -1, limit lower=-1 upper=1 effort=0 velocity=0
- added joint j_steering_f_r: type revolute, parent base_link, child steering_f_r, origin xyz=0.1135 -0.07475 0 rpy=0 -0.087266 0, axis 0 0 -1, limit lower=-1 upper=1 effort=0 velocity=0
- added joint j_tire_f_l: type continuous, parent steering_f_l, child tire_f_l, origin xyz=0 0 0 rpy=0 0.087266 0, axis 0 1 0
- added joint j_tire_f_r: type continuous, parent steering_f_r, child tire_f_r, origin xyz=0 0 0 rpy=0 0.087266 0, axis 0 1 0
- added joint j_tire_r_l: type continuous, parent base_link, child tire_r_l, origin xyz=-0.1135 0.07475 0 rpy=0 0 0, axis 0 1 0
- added joint j_tire_r_r: type continuous, parent base_link, child tire_r_r, origin xyz=-0.1135 -0.07475 0 rpy=0 0 0, axis 0 1 0

Commit message: urdf correction

File: ros_ws/src/description/urdf/description.urdf (robot description, URDF)
Before this commit: robot description, 8 links, 7 joints
Links:
- added link front_axle, mass 0
- added link rear_axle, mass 0
Joints:
- removed joint camera
- added joint j_camera: type fixed, parent base_link, child camera, origin xyz=0.0814 0 0.11015 rpy=0 0.17453 0, axis 0 0 0
- added joint j_front_axle: type fixed, parent base_link, child front_axle, origin xyz=0.1135 0 0 rpy=0 0 0, axis 0 0 0
- added joint j_rear_axle: type fixed, parent base_link, child rear_axle, origin xyz=-0.1135 0 0 rpy=0 0 0, axis 0 0 0
- joint j_steering_f_l: origin xyz=0.1135 0.07475 0 rpy=0 -0.087266 0 -> xyz=0.1135 0.07475 0 rpy=0 -0.0872664625997165 0
- joint j_tire_f_l: mimic (none) -> joint=j_tire_f_r multiplier=1 offset=0
- joint j_tire_f_r: axis 0 1 0 -> 0 -1 0; origin xyz=0 0 0 rpy=0 0.087266 0 -> xyz=0 0 0 rpy=0 0.0872664625997168 0
- joint j_tire_r_l: mimic (none) -> joint=j_tire_r_r multiplier=1 offset=0

Commit message: description change

File: ros_ws/src/description/urdf/description.urdf (robot description, URDF)
Before this commit: robot description, 10 links, 9 joints
Joints:
- joint j_camera: origin xyz=0.0814 0 0.11015 rpy=0 0.17453 0 -> xyz=0.0814000447600324 0.00875000004656613 0.110154914552125 rpy=0 0.174532925199437 0
- joint j_steering_f_r: origin xyz=0.1135 -0.07475 0 rpy=0 -0.087266 0 -> xyz=0.1135 -0.07475 0 rpy=0 -0.0872664625997168 0
- joint j_tire_f_l: origin xyz=0 0 0 rpy=0 0.087266 0 -> xyz=0 0 0 rpy=0 0.0872664625997165 0
